File: badgeelec.sch (KiCad schematic (older format))
At the start: 26 parts, among them J1 PROG_CONN, U1 PIC16F84A-XX/SO, U2 TSDP341xx

Commit message: prototype r1
Parts:
- removed JP2: reset, symbol Jumper_NO_Small
- added S1: PTS645SM43SMTR92, Buttons_Switches_SMD:SW_SPST_PTS645, symbol SPST
- BT1: footprint (none) -> 0gbadge-2018:BC-2003-TR
- C1, C2, C3: footprint (none) -> Capacitors_SMD:C_0805
- D1, D2, D3, D4, D5, D6, D7, D8: footprint LEDs:LED_0805_HandSoldering -> LEDs:LED_0805
- D10: footprint LEDs:LED_0805_HandSoldering -> LEDs:LED_1206
- D9: footprint LEDs:LED_0805_HandSoldering -> LEDs:LED_D3.0mm
- JP1: footprint (none) -> Oddities:NetTie-I_SMD
- U1: value PIC16F84A-XX/SO -> PIC16F716-I-SO-ND; footprint (none) -> Housings_SOIC:SOIC-18W_7.5x11.6mm_Pitch1.27mm
- U2: value TSDP341xx -> TSSP58038
Connections:
- wire segments 42 -> 43
Other:
- note added: "IR204\nNominal voltage: 1.2V\nPeak: 1A\nPeak WL: 940nm"
- note added: "Optional"
- note removed: "Not sure if I need this?"
- moved on the sheet: BT1
