File: badgeelec.sch (KiCad schematic (older format))
At the start: 26 parts, among them J1 PROG_CONN, U1 PIC16F716-I-SO-ND, U2 TSSP58038

Commit message: Halfway through v2
Parts:
- added C4, C5: 18pF, Capacitors_SMD:C_0805, symbol C_Small
- added Y1: 4Mhz, Crystals:Crystal_HC49-U_Vertical, symbol Crystal
- R7: value 1K -> 33K
Connections:
- net GND: now also C4.2, C5.2
- net at U1.15 (OSC2/CLKOUT): now also C5.1, Y1.2
- net at U1.16 (OSC1/CLKIN): now also C4.1, Y1.1
- no-connect marks 6 -> 4
Changed lines of the file:
@@
 $EndComp
 $Comp
-L VDD #PWR01
+L VDD #PWR8
 U 1 1 5A99BD61
 P 3400 2550
-F 0 "#PWR01" H 3400 2400 50  0001 C CNN
+F 0 "#PWR8" H 3400 2400 50  0001 C CNN
 F 1 "VDD" H 3400 2700 50  0000 C CNN
 F 2 "" H 3400 2550 50  0001 C CNN
@@
 $EndComp
 $Comp
-L GND #PWR02
+L GND #PWR9
 U 1 1 5A99BD79
 P 3400 4950
-F 0 "#PWR02" H 3400 4700 50  0001 C CNN
+F 0 "#PWR9" H 3400 4700 50  0001 C CNN
 F 1 "GND" H 3400 4800 50  0000 C CNN
 F 2 "" H 3400 4950 50  0001 C CNN
@@
 $EndComp
 $Comp
-L GND #PWR03
+L GND #PWR18
 U 1 1 5A99BEAA
 P 8650 1700
-F 0 "#PWR03" H 8650 1450 50  0001 C CNN
+F 0 "#PWR18" H 8650 1450 50  0001 C CNN
 F 1 "GND" H 8650 1550 50  0000 C CNN
 F 2 "" H 8650 1700 50  0001 C CNN
@@
 $EndComp
 $Comp
-L VDD #PWR04
+L VDD #PWR17
 U 1 1 5A99BFEB
 P 8650 1150
-F 0 "#PWR04" H 8650 1000 50  0001 C CNN
+F 0 "#PWR17" H 8650 1000 50  0001 C CNN
 F 1 "VDD" H 8650 1300 50  0000 C CNN
 F 2 "" H 8650 1150 50  0001 C CNN
@@
 $EndComp
 $Comp
-L VDD #PWR05
+L VDD #PWR1
 U 1 1 5A99C0C7
 P 1575 1075
-F 0 "#PWR05" H 1575 925 50  0001 C CNN
+F 0 "#PWR1" H 1575 925 50  0001 C CNN
 F 1 "VDD" H 1575 1225 50  0000 C CNN
 F 2 "" H 1575 1075 50  0001 C CNN
@@
 $EndComp
 $Comp
-L GND #PWR06
+L GND #PWR2
 U 1 1 5A99C10E
 P 1575 1375
-F 0 "#PWR06" H 1575 1125 50  0001 C CNN
+F 0 "#PWR2" H 1575 1125 50  0001 C CNN
 F 1 "GND" H 1575 1225 50  0000 C CNN
 F 2 "" H 1575 1375 50  0001 C CNN
@@
 $EndComp
 $Comp
-L PWR_FLAG #FLG07
+L PWR_FLAG #FLG1
 U 1 1 5A99C1B6
 P 1575 1075
-F 0 "#FLG07" H 1575 1150 50  0001 C CNN
+F 0 "#FLG1" H 1575 1150 50  0001 C CNN
 F 1 "PWR_FLAG" V 1575 1375 50  0000 C CNN
 F 2 "" H 1575 1075 50  0001 C CNN
@@
 $EndComp
 $Comp
-L PWR_FLAG #FLG08
+L PWR_FLAG #FLG2
 U 1 1 5A99C1D7
 P 1575 1375
-F 0 "#FLG08" H 1575 1450 50  0001 C CNN
+F 0 "#FLG2" H 1575 1450 50  0001 C CNN
 F 1 "PWR_FLAG" V 1575 1675 50  0000 C CNN
 F 2 "" H 1575 1375 50  0001 C CNN
@@
 $EndComp
 $Comp
-L GND #PWR09
+L GND #PWR13
 U 1 1 5A9DB86D
 P 4700 3650
-F 0 "#PWR09" H 4700 3400 50  0001 C CNN
+F 0 "#PWR13" H 4700 3400 50  0001 C CNN
 F 1 "GND" H 4700 3500 50  0000 C CNN
 F 2 "" H 4700 3650 50  0001 C CNN
@@
 $EndComp
 $Comp
-L VDD #PWR010
+L VDD #PWR14
 U 1 1 5A9DB88A
 P 4700 4050
-F 0 "#PWR010" H 4700 3900 50  0001 C CNN
+F 0 "#PWR14" H 4700 3900 50  0001 C CNN
 F 1 "VDD" H 4700 4200 50  0000 C CNN
 F 2 "" H 4700 4050 50  0001 C CNN
@@
 $EndComp
 $Comp
-L GND #PWR011
+L GND #PWR11
 U 1 1 5A9F157E
 P 4400 1250
-F 0 "#PWR011" H 4400 1000 50  0001 C CNN
+F 0 "#PWR11" H 4400 1000 50  0001 C CNN
 F 1 "GND" V 4400 1050 50  0000 C CNN
 F 2 "" H 4400 1250 50  0001 C CNN
@@
 ~MCLR
 $Comp
-L VDD #PWR012
+L VDD #PWR10
 U 1 1 5A9F163B
 P 4400 1150
-F 0 "#PWR012" H 4400 1000 50  0001 C CNN
+F 0 "#PWR10" H 4400 1000 50  0001 C CNN
 F 1 "VDD" V 4400 1350 50  0000 C CNN
 F 2 "" H 4400 1150 50  0001 C CNN
@@
 $EndComp
 $Comp
-L GND #PWR013
+L GND #PWR20
 U 1 1 5A9F1F88
 P 8650 2900
-F 0 "#PWR013" H 8650 2650 50  0001 C CNN
+F 0 "#PWR20" H 8650 2650 50  0001 C CNN
 F 1 "GND" H 8650 2750 50  0000 C CNN
 F 2 "" H 8650 2900 50  0001 C CNN
@@
 $EndComp
 $Comp
-L VDD #PWR014
+L VDD #PWR19
 U 1 1 5A9F1F96
 P 8650 2350
-F 0 "#PWR014" H 8650 2200 50  0001 C CNN
+F 0 "#PWR19" H 8650 2200 50  0001 C CNN
 F 1 "VDD" H 8650 2500 50  0000 C CNN
 F 2 "" H 8650 2350 50  0001 C CNN
@@
 $EndComp
 $Comp
-L GND #PWR015
+L GND #PWR22
 U 1 1 5A9F2871
 P 10800 1700
-F 0 "#PWR015" H 10800 1450 50  0001 C CNN
+F 0 "#PWR22" H 10800 1450 50  0001 C CNN
 F 1 "GND" H 10800 1550 50  0000 C CNN
 F 2 "" H 10800 1700 50  0001 C CNN
@@
 $EndComp
 $Comp
-L VDD #PWR016
+L VDD #PWR21
 U 1 1 5A9F287F
 P 10800 1150
-F 0 "#PWR016" H 10800 1000 50  0001 C CNN
+F 0 "#PWR21" H 10800 1000 50  0001 C CNN
 F 1 "VDD" H 10800 1300 50  0000 C CNN
 F 2 "" H 10800 1150 50  0001 C CNN
@@
 $EndComp
 $Comp
-L GND #PWR017
+L GND #PWR24
 U 1 1 5A9F2897
 P 10800 2900
-F 0 "#PWR017" H 10800 2650 50  0001 C CNN
+F 0 "#PWR24" H 10800 2650 50  0001 C CNN
 F 1 "GND" H 10800 2750 50  0000 C CNN
 F 2 "" H 10800 2900 50  0001 C CNN
@@
 $EndComp
 $Comp
-L VDD #PWR018
+L VDD #PWR23
 U 1 1 5A9F28A5
 P 10800 2350
-F 0 "#PWR018" H 10800 2200 50  0001 C CNN
+F 0 "#PWR23" H 10800 2200 50  0001 C CNN
 F 1 "VDD" H 10800 2500 50  0000 C CNN
 F 2 "" H 10800 2350 50  0001 C CNN
@@
 Text Label 9800 2800 2    60   ~ 0
 RA3
-NoConn ~ 2700 3300
-NoConn ~ 2700 3500
 NoConn ~ 4100 3500
 $Comp
@@
 P 2950 1200
 F 0 "R7" H 3050 1200 50  0000 C CNN
-F 1 "1K" V 2950 1200 50  0000 C CNN
+F 1 "33K" V 2950 1200 50  0000 C CNN
 F 2 "Resistors_SMD:R_0805_HandSoldering" V 2880 1200 50  0001 C CNN
 F 3 "" H 2950 1200 50  0001 C CNN
@@
 $EndComp
 $Comp
-L VDD #PWR019
+L VDD #PWR7
 U 1 1 5A9F3F17
 P 2950 1050
-F 0 "#PWR019" H 2950 900 50  0001 C CNN
+F 0 "#PWR7" H 2950 900 50  0001 C CNN
 F 1 "VDD" H 2950 1200 50  0000 C CNN
 F 2 "" H 2950 1050 50  0001 C CNN
@@
 $EndComp
 $Comp
-L GND #PWR020
+L GND #PWR6
 U 1 1 5A9F4B3B
 P 2800 2000
-F 0 "#PWR020" H 2800 1750 50  0001 C CNN
+F 0 "#PWR6" H 2800 1750 50  0001 C CNN
 F 1 "GND" H 2800 1850 50  0000 C CNN
 F 2 "" H 2800 2000 50  0001 C CNN
@@
 $EndComp
 $Comp
-L GND #PWR021
+L GND #PWR15
 U 1 1 5A9F5900
 P 5900 2000
-F 0 "#PWR021" H 5900 1750 50  0001 C CNN
+F 0 "#PWR15" H 5900 1750 50  0001 C CNN
 F 1 "GND" H 5900 1850 50  0000 C CNN
 F 2 "" H 5900 2000 50  0001 C CNN
@@
 $EndComp
 $Comp
-L GND #PWR022
+L GND #PWR16
 U 1 1 5A9F66F5
 P 6150 4400
-F 0 "#PWR022" H 6150 4150 50  0001 C CNN
+F 0 "#PWR16" H 6150 4150 50  0001 C CNN
 F 1 "GND" H 6150 4250 50  0000 C CNN
 F 2 "" H 6150 4400 50  0001 C CNN
@@
 NoConn ~ 4100 4200
 $Comp
-L GND #PWR023
+L GND #PWR4
 U 1 1 5A9F7413
 P 2400 2000
-F 0 "#PWR023" H 2400 1750 50  0001 C CNN
+F 0 "#PWR4" H 2400 1750 50  0001 C CNN
 F 1 "GND" H 2400 1850 50  0000 C CNN
 F 2 "" H 2400 2000 50  0001 C CNN
@@
 	2950 1350 2950 1450
 Wire Wire Line
-	2950 1650 2950 1800
+	2950 1800 2950 1650
 Wire Wire Line
 	2700 1800 3050 1800
@@
 Connection ~ 4100 2800
 $Comp
-L GND #PWR?
+L GND #PWR12
 U 1 1 5AA314FE
 P 4525 2800
-F 0 "#PWR?" H 4525 2550 50  0001 C CNN
+F 0 "#PWR12" H 4525 2550 50  0001 C CNN
 F 1 "GND" H 4525 2650 50  0000 C CNN
 F 2 "" H 4525 2800 50  0001 C CNN
@@
 	1    0    0    -1
 $EndComp
+$Comp
+L Crystal Y1
+U 1 1 5AC659A2
+P 2300 3850
+F 0 "Y1" H 2300 4000 50  0000 C CNN
+F 1 "4Mhz" H 2300 3700 50  0000 C CNN
+F 2 "Crystals:Crystal_HC49-U_Vertical" H 2300 3850 50  0001 C CNN
+F 3 "" H 2300 3850 50  0001 C CNN
+	1    2300 3850
+	1    0    0    -1
+$EndComp
+Wire Wire Line
+	2700 3300 2150 3300
+Wire Wire Line
+	2150 3300 2150 3850
+Wire Wire Line
+	2450 3850 2450 3500
+Wire Wire Line
+	2450 3500 2700 3500
+$Comp
+L C_Small C4
+U 1 1 5AC65CE6
+P 1950 4150
+F 0 "C4" H 1960 4220 50  0000 L CNN
+F 1 "18pF" H 1960 4070 50  0000 L CNN
+F 2 "Capacitors_SMD:C_0805" H 1950 4150 50  0001 C CNN
+F 3 "" H 1950 4150 50  0001 C CNN
+	1    1950 4150
+	1    0    0    -1
+$EndComp
+$Comp
+L C_Small C5
+U 1 1 5AC65D7C
+P 2650 4150
+F 0 "C5" H 2660 4220 50  0000 L CNN
+F 1 "18pF" H 2660 4070 50  0000 L CNN
+F 2 "Capacitors_SMD:C_0805" H 2650 4150 50  0001 C CNN
+F 3 "" H 2650 4150 50  0001 C CNN
+	1    2650 4150
+	1    0    0    -1
+$EndComp
+Wire Wire Line
+	1950 4050 1950 3850
+Wire Wire Line
+	1950 3850 2150 3850
+Wire Wire Line
+	2450 3850 2650 3850
+Wire Wire Line
+	2650 3850 2650 4050
+$Comp
+L GND #PWR5
+U 1 1 5AC65F49
+P 2650 4250
+F 0 "#PWR5" H 2650 4000 50  0001 C CNN
+F 1 "GND" H 2650 4100 50  0000 C CNN
+F 2 "" H 2650 4250 50  0001 C CNN
+F 3 "" H 2650 4250 50  0001 C CNN
+	1    2650 4250
+	1    0    0    -1
+$EndComp
+$Comp
+L GND #PWR3
+U 1 1 5AC66198
+P 1950 4250
+F 0 "#PWR3" H 1950 4000 50  0001 C CNN
+F 1 "GND" H 1950 4100 50  0000 C CNN
+F 2 "" H 1950 4250 50  0001 C CNN
+F 3 "" H 1950 4250 50  0001 C CNN
+	1    1950 4250
+	1    0    0    -1
+$EndComp

Commit message: Implemented prototypev2
Parts:
- removed JP1: permit operation / !program, Oddities:NetTie-I_SMD, symbol Jumper_NC_Small
- added J2: PWR_CONN, Pin_Headers:Pin_Header_Straight_1x02_Pitch2.54mm, symbol CONN_01X02
- BT1: Digikey (none) -> https://www.digikey.com/product-detail/en/mpd-memory-protec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
- C1: Digikey (none) -> https://www.digikey.com/product-detail/en/samsung-electro-m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
- C2: value 4.7uF -> 1uF; Digikey (none) -> https://www.digikey.com/product-detail/en/yageo/CC0805KKX5R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
- C3: value 100nF -> 10nF; Digikey (none) -> https://www.digikey.com/product-detail/en/samsung-electro-m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
- C4, C5: Digikey (none) -> https://www.digikey.com/product-detail/en/johanson-dielectr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
- R7: Digikey (none) -> https://www.digikey.com/product-detail/en/yageo/RC0805JR-07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
- U1: Digikey (none) -> https://www.digikey.com/product-detail/en/microchip-technol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
- U2: Digikey (none) -> https://www.digikey.com/product-detail/en/vishay-semiconduc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
- Y1: footprint Crystals:Crystal_HC49-U_Vertical -> 0gbadge-2018:ABLS-4MHZ-B2-T; Digikey (none) -> https://www.digikey.com/product-detail/en/abracon-llc/ABLS-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
Connections:
- net GND: now also J2.1 (P1)
- net VDD: now also J2.2 (P2)
- net ~MCLR: now also R7.2
Other:
- note added: "NOTE:\nNot likely to be populated / used\nfor attendee boards"
- note removed: "Internal OSC @ 4Mhz ( == 0.5mA?)"

Commit message: Schematic for final layout prototype 1
Parts:
- removed D10: LED, LEDs:LED_1206, symbol LED
- removed R6: 220, Resistors_SMD:R_0805_HandSoldering, symbol R
Connections:
- no-connect marks 4 -> 5
Other:
- note added: "Green-Blue RIGHT"
- note added: "Lower number designator = LEFT (except D3)"
- note added: "Orange/Yellow LEFT RIGHT"
- note added: "Red LEFT RIGHT"
- note removed: "Backlight 'G' LED"
- note removed: "Red-Orange LEFT"
- note removed: "Red-Orange RIGHT"
Changed lines of the file:
@@
 RB1
 Text Notes 7650 1850 0    60   ~ 0
-Red-Orange LEFT
+Red LEFT RIGHT
 $Comp
 L LED D4
@@
 	1    0    0    -1
 $EndComp
-Text Notes 9800 1850 0    60   ~ 0
-Red-Orange RIGHT
+Text Notes 9450 1850 0    60   ~ 0
+Orange/Yellow LEFT RIGHT
 $Comp
 L LED D8
@@
 $EndComp
 Text Notes 9800 3050 0    60   ~ 0
-Green-Blue LEFT
+Green-Blue RIGHT
 Text Label 4100 3100 0    60   ~ 0
 RA0
@@
 Optional
 $Comp
-L LED D10
-U 1 1 5A9F52D5
-P 6350 2000
-F 0 "D10" H 6350 2100 50  0000 C CNN
-F 1 "LED" H 6350 1900 50  0000 C CNN
-F 2 "LEDs:LED_1206" H 6350 2000 50  0001 C CNN
-F 3 "http://www.inolux-corp.com/datasheet/SMDLED/Mono%20Color%20Reverse%20Mount/IN-S124BR%20Series_V1.0.pdf" H 6350 2000 50  0001 C CNN
-	1    6350 2000
-	1    0    0    -1
-$EndComp
-$Comp
-L R R6
-U 1 1 5A9F536A
-P 6050 2000
-F 0 "R6" V 6130 2000 50  0000 C CNN
-F 1 "220" V 6050 2000 50  0000 C CNN
-F 2 "Resistors_SMD:R_0805_HandSoldering" V 5980 2000 50  0001 C CNN
-F 3 "" H 6050 2000 50  0001 C CNN
-	1    6050 2000
-	0    1    1    0
-$EndComp
-$Comp
-L GND #PWR021
-U 1 1 5A9F5900
-P 5900 2000
-F 0 "#PWR021" H 5900 1750 50  0001 C CNN
-F 1 "GND" H 5900 1850 50  0000 C CNN
-F 2 "" H 5900 2000 50  0001 C CNN
-F 3 "" H 5900 2000 50  0001 C CNN
-	1    5900 2000
-	1    0    0    -1
-$EndComp
-Text Label 6500 2000 0    60   ~ 0
-RB1
-Text Notes 6100 2200 0    60   ~ 0
-Backlight 'G' LED
-$Comp
 L R R8
 U 1 1 5A9F61AD
@@
 $EndComp
 $Comp
-L GND #PWR022
+L GND #PWR021
 U 1 1 5A9F66F5
 P 6150 4400
-F 0 "#PWR022" H 6150 4150 50  0001 C CNN
+F 0 "#PWR021" H 6150 4150 50  0001 C CNN
 F 1 "GND" H 6150 4250 50  0000 C CNN
 F 2 "" H 6150 4400 50  0001 C CNN
@@
 NoConn ~ 4100 4200
 $Comp
-L GND #PWR023
+L GND #PWR022
 U 1 1 5A9F7413
 P 2400 2000
-F 0 "#PWR023" H 2400 1750 50  0001 C CNN
+F 0 "#PWR022" H 2400 1750 50  0001 C CNN
 F 1 "GND" H 2400 1850 50  0000 C CNN
 F 2 "" H 2400 2000 50  0001 C CNN
@@
 Connection ~ 4100 2800
 $Comp
-L GND #PWR024
+L GND #PWR023
 U 1 1 5AA314FE
 P 4525 2800
-F 0 "#PWR024" H 4525 2550 50  0001 C CNN
+F 0 "#PWR023" H 4525 2550 50  0001 C CNN
 F 1 "GND" H 4525 2650 50  0000 C CNN
 F 2 "" H 4525 2800 50  0001 C CNN
@@
 	2650 3850 2650 4050
 $Comp
-L GND #PWR025
+L GND #PWR024
 U 1 1 5AC65F49
 P 2650 4250
-F 0 "#PWR025" H 2650 4000 50  0001 C CNN
+F 0 "#PWR024" H 2650 4000 50  0001 C CNN
 F 1 "GND" H 2650 4100 50  0000 C CNN
 F 2 "" H 2650 4250 50  0001 C CNN
@@
 $EndComp
 $Comp
-L GND #PWR026
+L GND #PWR025
 U 1 1 5AC66198
 P 1950 4250
-F 0 "#PWR026" H 1950 4000 50  0001 C CNN
+F 0 "#PWR025" H 1950 4000 50  0001 C CNN
 F 1 "GND" H 1950 4100 50  0000 C CNN
 F 2 "" H 1950 4250 50  0001 C CNN
@@
 $EndComp
 $Comp
-L GND #PWR027
+L GND #PWR026
 U 1 1 5ACBF8C3
 P 4650 1825
-F 0 "#PWR027" H 4650 1575 50  0001 C CNN
+F 0 "#PWR026" H 4650 1575 50  0001 C CNN
 F 1 "GND" V 4650 1625 50  0000 C CNN
 F 2 "" H 4650 1825 50  0001 C CNN
@@
 $EndComp
 $Comp
-L VDD #PWR028
+L VDD #PWR027
 U 1 1 5ACBF925
 P 4650 1925
-F 0 "#PWR028" H 4650 1775 50  0001 C CNN
+F 0 "#PWR027" H 4650 1775 50  0001 C CNN
 F 1 "VDD" V 4650 2125 50  0000 C CNN
 F 2 "" H 4650 1925 50  0001 C CNN
@@
 	0    -1   -1   0
 $EndComp
+Text Notes 8550 850  0    60   ~ 0
+Lower number designator = LEFT (except D3)
+NoConn ~ 4100 3800
 $EndSCHEMATC

Commit message: Created/changed IR receiver to horizontal footprint, implemented basic generator for poker-chip style layout
Parts:
- U2: footprint Opto-Devices:IRReceiver_Vishay_MOLD-3pin -> 0gbadge-2018:tssp58038_flat
Changed lines of the file:
@@
 F 0 "U2" H 4700 4150 50  0000 L CNN
 F 1 "TSSP58038" H 4700 3550 50  0000 L CNN
-F 2 "Opto-Devices:IRReceiver_Vishay_MOLD-3pin" H 5050 3475 50  0001 C CNN
+F 2 "0gbadge-2018:tssp58038_flat" H 5050 3475 50  0001 C CNN
 F 3 "http://www.vishay.com/docs/82479/tssp58038.pdf" H 5750 4150 50  0001 C CNN
 F 4 "https://www.digikey.com/product-detail/en/vishay-semiconductor-opto-division/TSSP58038/TSSP58038-ND/4695717" H 5100 3850 60  0001 C CNN "Digikey"

Commit message: Routed prototype final v1
Connections:
- net RA1: no longer R3.2
- net RB3: now also R3.2
Changed lines of the file:
@@
 Text Label 7650 1600 2    60   ~ 0
 RA0
-Text Label 7650 2800 2    60   ~ 0
-RA1
 Text Label 9800 1600 2    60   ~ 0
 RA2
@@
 	1    0    0    -1
 $EndComp
-NoConn ~ 4100 4000
+NoConn ~ 4100 3200
 NoConn ~ 4100 4100
 NoConn ~ 4100 4200
@@
 Lower number designator = LEFT (except D3)
 NoConn ~ 4100 3800
+Text Label 7650 2800 2    60   ~ 0
+RB3
 $EndSCHEMATC

Commit message: check in gerber zip
Other:
- note added: "Optional, probably not present"
Changed lines of the file:
@@
 Text Label 7650 2800 2    60   ~ 0
 RB3
+Text Notes 4650 2150 0    60   ~ 0
+Optional, probably not present
 $EndSCHEMATC

Commit message: Cut r4
Parts:
- J1: footprint Pin_Headers:Pin_Header_Straight_1x05_Pitch2.54mm -> ext_libs:SMD_PROG_5
Changed lines of the file:
@@
 F 0 "J1" H 4850 1550 50  0000 C CNN
 F 1 "PROG_CONN" H 4850 950 50  0000 C CNN
-F 2 "Pin_Headers:Pin_Header_Straight_1x05_Pitch2.54mm" H 4850 1250 50  0001 C CNN
+F 2 "ext_libs:SMD_PROG_5" H 4850 1250 50  0001 C CNN
 F 3 "" H 4850 1250 50  0001 C CNN
 	1    4850 1250

Commit message: First pass verifying everything
Parts:
- removed C3: 10nF, Capacitors_SMD:C_0805, symbol C_Small
- removed J2: PWR_CONN, Pin_Headers:Pin_Header_Straight_1x02_Pitch2.54mm, symbol CONN_01X02
- removed S1: PTS645SM43SMTR92, Buttons_Switches_SMD:SW_SPST_PTS645, symbol SPST
- R1: value 220 -> 1k
- R2: value 220 -> 430
- R3, R4: value 150 -> 220
- R8: value 200R -> 220
Other:
- note removed: "IR204\nNominal voltage: 1.2V\nPeak: 1A\nPeak WL: 940nm"
- note removed: "NOTE:\nNot likely to be populated / used\nfor attendee boards"
- note removed: "Optional"
- note removed: "Optional, probably not present"
Changed lines of the file:
@@
 encoding utf-8
 Sheet 1 1
-Title "LED prototype"
-Date "2018-04-09"
-Rev "2"
+Title "0x0G electronic badge"
+Date "2018-05-07"
+Rev "4"
 Comp "Google LLC"
-Comment1 "0xG prototype to test programming, IR, ICSP."
-Comment2 "External Crystal added, increased pullup value to 33k for ~MCLR"
-Comment3 "Added PWR_CONN for external power"
-Comment4 "Fix incorrect polarity on battery holder"
+Comment1 "Removed components that will not be on final board"
+Comment2 ""
+Comment3 ""
+Comment4 ""
 $EndDescr
 $Comp
@@
 P 7800 1600
 F 0 "R1" V 7880 1600 50  0000 C CNN
-F 1 "220" V 7800 1600 50  0000 C CNN
+F 1 "1k" V 7800 1600 50  0000 C CNN
 F 2 "Resistors_SMD:R_0805_HandSoldering" V 7730 1600 50  0001 C CNN
 F 3 "" H 7800 1600 50  0001 C CNN
@@
 P 7800 2800
 F 0 "R3" V 7880 2800 50  0000 C CNN
-F 1 "150" V 7800 2800 50  0000 C CNN
+F 1 "220" V 7800 2800 50  0000 C CNN
 F 2 "Resistors_SMD:R_0805_HandSoldering" V 7730 2800 50  0001 C CNN
 F 3 "" H 7800 2800 50  0001 C CNN
@@
 P 9950 1600
 F 0 "R2" V 10030 1600 50  0000 C CNN
-F 1 "220" V 9950 1600 50  0000 C CNN
+F 1 "430" V 9950 1600 50  0000 C CNN
 F 2 "Resistors_SMD:R_0805_HandSoldering" V 9880 1600 50  0001 C CNN
 F 3 "" H 9950 1600 50  0001 C CNN
@@
 P 9950 2800
 F 0 "R4" V 10030 2800 50  0000 C CNN
-F 1 "150" V 9950 2800 50  0000 C CNN
+F 1 "220" V 9950 2800 50  0000 C CNN
 F 2 "Resistors_SMD:R_0805_HandSoldering" V 9880 2800 50  0001 C CNN
 F 3 "" H 9950 2800 50  0001 C CNN
@@
 	1    0    0    -1
 $EndComp
-Text Label 3050 1800 0    60   ~ 0
+Text Label 2950 1800 0    60   ~ 0
 ~MCLR
-$Comp
-L C_Small C3
-U 1 1 5A9F4900
-P 2800 1900
-F 0 "C3" H 2810 1970 50  0000 L CNN
-F 1 "10nF" H 2810 1820 50  0000 L CNN
-F 2 "Capacitors_SMD:C_0805" H 2800 1900 50  0001 C CNN
-F 3 "" H 2800 1900 50  0001 C CNN
-F 4 "https://www.digikey.com/product-detail/en/samsung-electro-mechanics/CL21B102KBCNNNC/1276-2425-1-ND/3890511" H 2800 1900 60  0001 C CNN "Digikey"
-	1    2800 1900
-	1    0    0    -1
-$EndComp
-$Comp
-L GND #PWR020
-U 1 1 5A9F4B3B
-P 2800 2000
-F 0 "#PWR020" H 2800 1750 50  0001 C CNN
-F 1 "GND" H 2800 1850 50  0000 C CNN
-F 2 "" H 2800 2000 50  0001 C CNN
-F 3 "" H 2800 2000 50  0001 C CNN
-	1    2800 2000
-	1    0    0    -1
-$EndComp
-Text Notes 2850 2100 0    60   ~ 0
-Optional
 $Comp
 L R R8
@@
 P 6150 3950
 F 0 "R8" H 6250 3950 50  0000 C CNN
-F 1 "200R" V 6150 3950 50  0000 C CNN
+F 1 "220" V 6150 3950 50  0000 C CNN
 F 2 "Resistors_SMD:R_0805_HandSoldering" V 6080 3950 50  0001 C CNN
 F 3 "" H 6150 3950 50  0001 C CNN
@@
 $EndComp
 $Comp
-L GND #PWR021
+L GND #PWR020
 U 1 1 5A9F66F5
 P 6150 4400
-F 0 "#PWR021" H 6150 4150 50  0001 C CNN
+F 0 "#PWR020" H 6150 4150 50  0001 C CNN
 F 1 "GND" H 6150 4250 50  0000 C CNN
 F 2 "" H 6150 4400 50  0001 C CNN
@@
 NoConn ~ 4100 4100
 NoConn ~ 4100 4200
-$Comp
-L GND #PWR022
-U 1 1 5A9F7413
-P 2400 2000
-F 0 "#PWR022" H 2400 1750 50  0001 C CNN
-F 1 "GND" H 2400 1850 50  0000 C CNN
-F 2 "" H 2400 2000 50  0001 C CNN
-F 3 "" H 2400 2000 50  0001 C CNN
-	1    2400 2000
-	1    0    0    -1
-$EndComp
-$Comp
-L SPST S1
-U 1 1 5AA2DBC2
-P 2550 1800
-F 0 "S1" H 2540 1885 60  0000 C CNN
-F 1 "PTS645SM43SMTR92" H 1925 1750 60  0000 C CNN
-F 2 "Buttons_Switches_SMD:SW_SPST_PTS645" H 2550 1800 60  0001 C CNN
-F 3 "https://www.ckswitches.com/media/1471/pts645.pdf" H 2550 1800 60  0001 C CNN
-	1    2550 1800
-	1    0    0    -1
-$EndComp
 $Bitmap
 Pos 11125 7050
@@
 EndData
 $EndBitmap
-Text Notes 6250 4650 0    60   ~ 0
-IR204\nNominal voltage: 1.2V\nPeak: 1A\nPeak WL: 940nm
 Wire Wire Line
 	3400 4950 3400 4700
@@
 	2950 1350 2950 1800
 Wire Wire Line
-	2700 1800 3050 1800
-Connection ~ 2950 1800
-Connection ~ 2800 1800
-Wire Wire Line
-	2400 2000 2400 1800
-Wire Wire Line
 	3700 2750 3700 2800
 Wire Wire Line
@@
 Connection ~ 4100 2800
 $Comp
-L GND #PWR023
+L GND #PWR021
 U 1 1 5AA314FE
 P 4525 2800
-F 0 "#PWR023" H 4525 2550 50  0001 C CNN
+F 0 "#PWR021" H 4525 2550 50  0001 C CNN
 F 1 "GND" H 4525 2650 50  0000 C CNN
 F 2 "" H 4525 2800 50  0001 C CNN
@@
 	2650 3850 2650 4050
 $Comp
-L GND #PWR024
+L GND #PWR022
 U 1 1 5AC65F49
 P 2650 4250
-F 0 "#PWR024" H 2650 4000 50  0001 C CNN
+F 0 "#PWR022" H 2650 4000 50  0001 C CNN
 F 1 "GND" H 2650 4100 50  0000 C CNN
 F 2 "" H 2650 4250 50  0001 C CNN
@@
 $EndComp
 $Comp
-L GND #PWR025
+L GND #PWR023
 U 1 1 5AC66198
 P 1950 4250
-F 0 "#PWR025" H 1950 4000 50  0001 C CNN
+F 0 "#PWR023" H 1950 4000 50  0001 C CNN
 F 1 "GND" H 1950 4100 50  0000 C CNN
 F 2 "" H 1950 4250 50  0001 C CNN
@@
 	1    1950 4250
 	1    0    0    -1
-$EndComp
-Text Notes 6375 3900 0    60   ~ 12
-NOTE:\nNot likely to be populated / used\nfor attendee boards
-$Comp
-L CONN_01X02 J2
-U 1 1 5ACBF681
-P 4850 1875
-F 0 "J2" H 4850 2025 50  0000 C CNN
-F 1 "PWR_CONN" H 4850 1725 50  0000 C CNN
-F 2 "Pin_Headers:Pin_Header_Straight_1x02_Pitch2.54mm" H 4850 1875 50  0001 C CNN
-F 3 "" H 4850 1875 50  0001 C CNN
-	1    4850 1875
-	1    0    0    -1
-$EndComp
-$Comp
-L GND #PWR026
-U 1 1 5ACBF8C3
-P 4650 1825
-F 0 "#PWR026" H 4650 1575 50  0001 C CNN
-F 1 "GND" V 4650 1625 50  0000 C CNN
-F 2 "" H 4650 1825 50  0001 C CNN
-F 3 "" H 4650 1825 50  0001 C CNN
-	1    4650 1825
-	0    1    1    0
-$EndComp
-$Comp
-L VDD #PWR027
-U 1 1 5ACBF925
-P 4650 1925
-F 0 "#PWR027" H 4650 1775 50  0001 C CNN
-F 1 "VDD" V 4650 2125 50  0000 C CNN
-F 2 "" H 4650 1925 50  0001 C CNN
-F 3 "" H 4650 1925 50  0001 C CNN
-	1    4650 1925
-	0    -1   -1   0
 $EndComp
 Text Notes 8550 850  0    60   ~ 0
@@
 Text Label 7650 2800 2    60   ~ 0
 RB3
-Text Notes 4650 2150 0    60   ~ 0
-Optional, probably not present
 $EndSCHEMATC
