File: programmer/programmer.sch (KiCad schematic (older format))
At the start: 12 parts, among them J1 USB_A, J2 PWR, J3 PICKIT, J4 POGO_BOARD, J5 TEST_2P

Commit message: Update programmer
Parts:
- removed J1: USB_A, Connect:USB_A, symbol USB_A
- added J1: USB_OTG, Connector_USB:USB_Micro-B_Amphenol_10103594-0001LF_Horizontal, symbol USB_OTG
- J4: footprint prog:SMD-5 -> Pin_Headers:Pin_Header_Straight_1x05_Pitch2.54mm
Connections:
- net GND: now also J1.5 (GND)
- net at R1.2, R2.2: now also J1.1 (VBUS)
- no-connect marks 4 -> 5
Changed lines of the file:
@@
 F 0 "J4" H 8100 3050 50  0000 C CNN
 F 1 "POGO_BOARD" V 8200 2750 50  0000 C CNN
-F 2 "prog:SMD-5" H 8100 2750 50  0001 C CNN
+F 2 "Pin_Headers:Pin_Header_Straight_1x05_Pitch2.54mm" H 8100 2750 50  0001 C CNN
 F 3 "" H 8100 2750 50  0001 C CNN
 	1    8100 2750
@@
 Text Label 7700 2950 0    60   ~ 0
 PGC
-$Comp
-L USB_A J1
-U 1 1 5AF34ABD
-P 4750 2100
-F 0 "J1" H 4550 2550 50  0000 L CNN
-F 1 "USB_A" H 4550 2450 50  0000 L CNN
-F 2 "Connect:USB_A" H 4900 2050 50  0001 C CNN
-F 3 "" H 4900 2050 50  0001 C CNN
-	1    4750 2100
-	1    0    0    -1
-$EndComp
 NoConn ~ 4650 2500
 $Comp
@@
 Wire Wire Line
 	8100 3500 8100 3400
+$Comp
+L USB_OTG J1
+U 1 1 5AF372B9
+P 4750 2100
+F 0 "J1" H 4550 2550 50  0000 L CNN
+F 1 "USB_OTG" H 4550 2450 50  0000 L CNN
+F 2 "Connector_USB:USB_Micro-B_Amphenol_10103594-0001LF_Horizontal" H 4900 2050 50  0001 C CNN
+F 3 "" H 4900 2050 50  0001 C CNN
+	1    4750 2100
+	1    0    0    -1
+$EndComp
+NoConn ~ 5050 2300
 $EndSCHEMATC
